File: OpenWatts.kicad_sch (KiCad schematic)
At the start: 36 parts, among them J1 USB_C_Receptacle_USB2.0_16P, J2 Conn_02x03_Odd_Even, SW1 SW_Push, SW2 SW_Push, U1 MCP73831-2-OT, U2 ME6211C33M5, U4 HX711, U5 ESP32-C3-MINI-1, U6 LSM6DS3

Commit message: Checkpoint OpenWatts motion-wake firmware and board outputs
Parts:
- D2: value LED -> LED_RED
- D3: value LED -> LED_OTHER
Changed lines of the file:
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@@
 			)
 		)
-		(property "Value" "LED"
+		(property "Value" "LED_RED"
 			(at 61.9125 68.58 0)
 			(show_name no)
@@
 			)
 		)
-		(property "Value" "LED"
+		(property "Value" "LED_OTHER"
 			(at 61.9125 78.74 0)
 			(show_name no)

Commit message: Present OpenWatts RevA for public release
- Add a concise public README and human-readable RevA BOM
- Polish the schematic with functional headings and manufactured-board metadata
- Add PDF, SVG, front, back, and 3D public hardware assets
- Preserve evidence-based future hardware lessons in isolated RevB notes
- Remove local KiCad sessions, redundant exports, and unused artwork
- Keep the manufactured PCB and electrical connectivity unchanged
Other:
- note added: "BATTERY / USB SENSE & STATUS"
- note added: "ESP32-C3, USB & SERVICE I/O"
- note added: "IMU & MOTION SENSING"
- note added: "LiPo CHARGING & 3.3 V POWER"
- note added: "STRAIN BRIDGE & HX711"
- note added: "USB-C INPUT"
- company: (none) -> OpenWatts
- title: (none) -> OpenWatts Cycling Power Meter
Changed lines of the file:
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@@
 	(generator_version "10.0")
 	(paper "A4")
+	(title_block
+		(title "OpenWatts Cycling Power Meter")
+		(date "2026-07-06")
+		(rev "RevA")
+		(company "OpenWatts")
+		(comment 1 "Manufactured and field-validated hardware revision")
+		(comment 2 "ESP32-C3 / HX711 strain measurement / LSM6DS3 cadence")
+	)
+	(text "USB-C INPUT"
+		(at 17.78 17.78 0)
+		(effects (font (size 1.778 1.778) (bold yes)) (justify left bottom))
+	)
+	(text "LiPo CHARGING & 3.3 V POWER"
+		(at 76.2 17.78 0)
+		(effects (font (size 1.778 1.778) (bold yes)) (justify left bottom))
+	)
+	(text "ESP32-C3, USB & SERVICE I/O"
+		(at 137.16 17.78 0)
+		(effects (font (size 1.778 1.778) (bold yes)) (justify left bottom))
+	)
+	(text "STRAIN BRIDGE & HX711"
+		(at 17.78 96.52 0)
+		(effects (font (size 1.778 1.778) (bold yes)) (justify left bottom))
+	)
+	(text "IMU & MOTION SENSING"
+		(at 88.9 96.52 0)
+		(effects (font (size 1.778 1.778) (bold yes)) (justify left bottom))
+	)
+	(text "BATTERY / USB SENSE & STATUS"
+		(at 111.76 76.2 0)
+		(effects (font (size 1.524 1.524) (bold yes)) (justify left bottom))
+	)
 	(junction
 		(at 46.99 41.91)
